File: esp32controller.kicad_pcb (KiCad board)
At the start: 2 copper layers, 31 x 26 mm, 16 parts, among them J1 DE9_Socket, Q1 AO3400A, Q2 AO3400A, Q3 AO3400A, Q4 AO3400A, Q5 AO3400A, Q6 AO3400A, Q7 AO3400A

Commit message: Added firmware, cleaned files
Routing:
- net +5V: track 0.00 -> 34.4 mm, vias 0 -> 1
- net GND: track 0.00 -> 13.9 mm, vias 0 -> 1
- added copper zone on B.Cu, net GND
Other:
- board size 31 x 26 mm -> 30.4 x 25.4 mm
Changed lines of the file:
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@@
 	)
 	(gr_rect
-		(start 156 82)
-		(end 187 108)
+		(start 156.6 82.4)
+		(end 187 107.8)
 		(stroke
 			(width 0.05)
@@
 	)
 	(segment
+		(start 162.38 89.38)
+		(end 162.38 86.11)
+		(width 0.4)
+		(layer "F.Cu")
+		(net 4)
+	)
+	(segment
+		(start 166.2 91)
+		(end 165.4 90.2)
+		(width 0.4)
+		(layer "F.Cu")
+		(net 4)
+	)
+	(segment
+		(start 165.4 90.2)
+		(end 163.2 90.2)
+		(width 0.4)
+		(layer "F.Cu")
+		(net 4)
+	)
+	(segment
+		(start 166.2 92.8)
+		(end 166.2 91)
+		(width 0.4)
+		(layer "F.Cu")
+		(net 4)
+	)
+	(segment
+		(start 163.2 90.2)
+		(end 162.38 89.38)
+		(width 0.4)
+		(layer "F.Cu")
+		(net 4)
+	)
+	(via
+		(at 166.2 92.8)
+		(size 0.6)
+		(drill 0.3)
+		(layers "F.Cu" "B.Cu")
+		(net 4)
+	)
+	(segment
+		(start 179.0625 90.05)
+		(end 177.125 90.05)
+		(width 0.4)
+		(layer "B.Cu")
+		(net 4)
+	)
+	(segment
+		(start 165 92.8)
+		(end 166.2 92.8)
+		(width 0.4)
+		(layer "B.Cu")
+		(net 4)
+	)
+	(segment
+		(start 177.125 90.05)
+		(end 177 90.175)
+		(width 0.4)
+		(layer "B.Cu")
+		(net 4)
+	)
+	(segment
+		(start 165 91.825)
+		(end 165 92.8)
+		(width 0.4)
+		(layer "B.Cu")
+		(net 4)
+	)
+	(segment
+		(start 159.2 91.2)
+		(end 159.84 90.56)
+		(width 0.6)
+		(layer "F.Cu")
+		(net 7)
+	)
+	(segment
+		(start 160.6 94.8)
+		(end 159.2 93.4)
+		(width 0.6)
+		(layer "F.Cu")
+		(net 7)
+	)
+	(segment
+		(start 159.2 93.4)
+		(end 159.2 91.2)
+		(width 0.6)
+		(layer "F.Cu")
+		(net 7)
+	)
+	(segment
+		(start 182 93.6)
+		(end 174.4 93.6)
+		(width 0.6)
+		(layer "F.Cu")
+		(net 7)
+	)
+	(segment
+		(start 159.84 90.56)
+		(end 159.84 86.11)
+		(width 0.6)
+		(layer "F.Cu")
+		(net 7)
+	)
+	(segment
+		(start 174.4 93.6)
+		(end 173.2 94.8)
+		(width 0.6)
+		(layer "F.Cu")
+		(net 7)
+	)
+	(segment
+		(start 173.2 94.8)
+		(end 160.6 94.8)
+		(width 0.6)
+		(layer "F.Cu")
+		(net 7)
+	)
+	(via
+		(at 182 93.6)
+		(size 0.6)
+		(drill 0.3)
+		(layers "F.Cu" "B.Cu")
+		(net 7)
+	)
+	(segment
+		(start 182.015 93.615)
+		(end 182 93.6)
+		(width 0.4)
+		(layer "B.Cu")
+		(net 7)
+	)
+	(segment
+		(start 185 93.615)
+		(end 182.015 93.615)
+		(width 0.6)
+		(layer "B.Cu")
+		(net 7)
+	)
+	(segment
 		(start 167.2 91.8)
 		(end 169.54 89.46)
@@
 	)
 	(segment
+		(start 160.2 93)
+		(end 160.8 93.6)
+		(width 0.4)
+		(layer "F.Cu")
+		(net 16)
+	)
+	(segment
+		(start 172.4 93.6)
+		(end 173.8 92.2)
+		(width 0.4)
+		(layer "F.Cu")
+		(net 16)
+	)
+	(segment
+		(start 173.8 92.2)
+		(end 173.83 92.23)
+		(width 0.4)
+		(layer "F.Cu")
+		(net 16)
+	)
+	(segment
+		(start 160.2 92.4)
+		(end 160.2 93)
+		(width 0.4)
+		(layer "F.Cu")
+		(net 16)
+	)
+	(segment
 		(start 160.8 93.6)
 		(end 172.4 93.6)
@@
 	)
 	(segment
-		(start 173.8 92.2)
-		(end 173.83 92.23)
-		(width 0.4)
-		(layer "F.Cu")
-		(net 16)
-	)
-	(segment
 		(start 173.83 92.23)
 		(end 185 92.23)
@@
 		(net 16)
 	)
-	(segment
-		(start 172.4 93.6)
-		(end 173.8 92.2)
-		(width 0.4)
-		(layer "F.Cu")
-		(net 16)
-	)
-	(segment
-		(start 159.6 92.4)
-		(end 160.8 93.6)
-		(width 0.4)
-		(layer "F.Cu")
-		(net 16)
-	)
 	(via
-		(at 159.6 92.4)
+		(at 160.2 92.4)
 		(size 0.6)
 		(drill 0.3)
@@
 	)
 	(segment
-		(start 161.0625 91)
+		(start 160.2 91.8)
 		(end 161 91)
 		(width 0.4)
@@
 	(segment
 		(start 161 91)
-		(end 159.6 92.4)
+		(end 161.0625 91)
+		(width 0.4)
+		(layer "B.Cu")
+		(net 16)
+	)
+	(segment
+		(start 160.2 92.4)
+		(end 160.2 91.8)
 		(width 0.4)
 		(layer "B.Cu")
@@
 		(net 24)
 	)
+	(zone
+		(net 4)
+		(net_name "GND")
+		(layer "B.Cu")
+		(hatch edge 0.5)
+		(connect_pads
+			(clearance 0.5)
+		)
+		(min_thickness 0.25)
+		(filled_areas_thickness no)
+		(fill yes
+			(thermal_gap 0.5)
+			(thermal_bridge_width 0.5)
+		)
+		(polygon
+			(pts
+				(xy 156.6 82.4) (xy 156.6 107.8) (xy 187 107.8) (xy 187 82.4)
+			)
+		)
+	)
 	(group ""

Commit message: Fixes to kicad files
Parts:
- e1: renamed from IC1; footprint bionik:ESP32S3_supermini -> project_parts:ESP32S3_supermini

Commit message: Updates to pcb
Parts:
- renumbered e1 to ESP32s3
Changed lines of the file:
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@@
 		(layer "F.Cu")
 		(at 170 95 90)
-		(property "Reference" "e1"
+		(property "Reference" "ESP32s3"
 			(at 0 -0.5 90)
 			(unlocked yes)
@@
 			(layers "*.Cu" "*.Mask")
 			(remove_unused_layers no)
-			(net "unconnected-(e1-TX-Pad1)")
+			(net "unconnected-(ESP32s3-TX-Pad1)")
 			(pinfunction "TX_1")
 			(pintype "input")
@@
 			(remove_unused_layers no)
 			(roundrect_rratio 0.15)
-			(net "unconnected-(e1-RX-Pad2)")
+			(net "unconnected-(ESP32s3-RX-Pad2)")
 			(pinfunction "RX_2")
 			(pintype "input")
@@
 			(remove_unused_layers no)
 			(roundrect_rratio 0.15)
-			(net "Net-(Q5-G)")
+			(net "Net-(ESP32s3-GPIO1)")
 			(pinfunction "GPIO1_3")
 			(pintype "input")
@@
 			(remove_unused_layers no)
 			(roundrect_rratio 0.15)
-			(net "unconnected-(e1-GPIO2-Pad4)")
+			(net "unconnected-(ESP32s3-GPIO2-Pad4)")
 			(pinfunction "GPIO2_4")
 			(pintype "input")
@@
 			(remove_unused_layers no)
 			(roundrect_rratio 0.15)
-			(net "Net-(Q7-G)")
+			(net "Net-(ESP32s3-GPIO3)")
 			(pinfunction "GPIO3_5")
 			(pintype "input")
@@
 			(remove_unused_layers no)
 			(roundrect_rratio 0.15)
-			(net "unconnected-(e1-GPIO4-Pad6)")
+			(net "unconnected-(ESP32s3-GPIO4-Pad6)")
 			(pinfunction "GPIO4_6")
 			(pintype "input")
@@
 			(remove_unused_layers no)
 			(roundrect_rratio 0.15)
-			(net "unconnected-(e1-GPIO5-Pad7)")
+			(net "unconnected-(ESP32s3-GPIO5-Pad7)")
 			(pinfunction "GPIO5_7")
 			(pintype "input")
@@
 			(remove_unused_layers no)
 			(roundrect_rratio 0.15)
-			(net "unconnected-(e1-GPIO6-Pad8)")
+			(net "unconnected-(ESP32s3-GPIO6-Pad8)")
 			(pinfunction "GPIO6_8")
 			(pintype "input")
@@
 			(remove_unused_layers no)
 			(roundrect_rratio 0.15)
-			(net "Net-(Q6-G)")
+			(net "Net-(ESP32s3-GPIO7)")
 			(pinfunction "GPIO7_9")
 			(pintype "input")
@@
 			(remove_unused_layers no)
 			(roundrect_rratio 0.15)
-			(net "unconnected-(e1-GPIO8-Pad10)")
+			(net "unconnected-(ESP32s3-GPIO8-Pad10)")
 			(pinfunction "GPIO8_10")
 			(pintype "input")
@@
 			(remove_unused_layers no)
 			(roundrect_rratio 0.15)
-			(net "Net-(Q2-G)")
+			(net "Net-(ESP32s3-GPIO9)")
 			(pinfunction "GPIO9_11")
 			(pintype "input")
@@
 			(remove_unused_layers no)
 			(roundrect_rratio 0.15)
-			(net "Net-(Q4-G)")
+			(net "Net-(ESP32s3-GPIO10)")
 			(pinfunction "GPIO10_12")
 			(pintype "input")
@@
 			(remove_unused_layers no)
 			(roundrect_rratio 0.15)
-			(net "Net-(Q1-G)")
+			(net "Net-(ESP32s3-GPIO11)")
 			(pinfunction "GPIO11_13")
 			(pintype "input")
@@
 			(remove_unused_layers no)
 			(roundrect_rratio 0.15)
-			(net "unconnected-(e1-GPIO12-Pad14)")
+			(net "unconnected-(ESP32s3-GPIO12-Pad14)")
 			(pinfunction "GPIO12_14")
 			(pintype "input")
@@
 			(remove_unused_layers no)
 			(roundrect_rratio 0.15)
-			(net "Net-(Q3-G)")
+			(net "Net-(ESP32s3-GPIO13)")
 			(pinfunction "GPIO13_15")
 			(pintype "input")
@@
 			(remove_unused_layers no)
 			(roundrect_rratio 0.15)
-			(net "unconnected-(e1-3V3-Pad16)")
+			(net "unconnected-(ESP32s3-3V3-Pad16)")
 			(pinfunction "3V3_16")
 			(pintype "input")
@@
 			(layers "B.Cu" "B.Mask" "B.Paste")
 			(roundrect_rratio 0.25)
-			(net "Net-(Q5-G)")
+			(net "Net-(ESP32s3-GPIO1)")
 			(pinfunction "G_1")
 			(pintype "input")
@@
 			(layers "B.Cu" "B.Mask" "B.Paste")
 			(roundrect_rratio 0.25)
-			(net "Net-(Q7-G)")
+			(net "Net-(ESP32s3-GPIO3)")
 			(pintype "passive")
 		)
@@
 			(layers "B.Cu" "B.Mask" "B.Paste")
 			(roundrect_rratio 0.25)
-			(net "Net-(Q6-G)")
+			(net "Net-(ESP32s3-GPIO7)")
 			(pinfunction "G_1")
 			(pintype "input")
@@
 			(layers "B.Cu" "B.Mask" "B.Paste")
 			(roundrect_rratio 0.25)
-			(net "Net-(Q7-G)")
+			(net "Net-(ESP32s3-GPIO3)")
 			(pinfunction "G_1")
 			(pintype "input")
@@
 			(layers "B.Cu" "B.Mask" "B.Paste")
 			(roundrect_rratio 0.25)
-			(net "Net-(Q2-G)")
+			(net "Net-(ESP32s3-GPIO9)")
 			(pinfunction "G_1")
 			(pintype "input")
@@
 			(layers "B.Cu" "B.Mask" "B.Paste")
 			(roundrect_rratio 0.25)
-			(net "Net-(Q3-G)")
+			(net "Net-(ESP32s3-GPIO13)")
 			(pinfunction "G_1")
 			(pintype "input")
@@
 			(layers "B.Cu" "B.Mask" "B.Paste")
 			(roundrect_rratio 0.25)
-			(net "Net-(Q4-G)")
+			(net "Net-(ESP32s3-GPIO10)")
 			(pinfunction "G_1")
 			(pintype "input")
@@
 			(layers "B.Cu" "B.Mask" "B.Paste")
 			(roundrect_rratio 0.25)
-			(net "Net-(Q3-G)")
+			(net "Net-(ESP32s3-GPIO13)")
 			(pintype "passive")
 		)
@@
 			(layers "B.Cu" "B.Mask" "B.Paste")
 			(roundrect_rratio 0.25)
-			(net "Net-(Q6-G)")
+			(net "Net-(ESP32s3-GPIO7)")
 			(pintype "passive")
 		)
@@
 			(layers "B.Cu" "B.Mask" "B.Paste")
 			(roundrect_rratio 0.25)
-			(net "Net-(Q1-G)")
+			(net "Net-(ESP32s3-GPIO11)")
 			(pintype "passive")
 		)
@@
 			(layers "B.Cu" "B.Mask" "B.Paste")
 			(roundrect_rratio 0.25)
-			(net "Net-(Q5-G)")
+			(net "Net-(ESP32s3-GPIO1)")
 			(pintype "passive")
 		)
@@
 			(layers "B.Cu" "B.Mask" "B.Paste")
 			(roundrect_rratio 0.25)
-			(net "Net-(Q4-G)")
+			(net "Net-(ESP32s3-GPIO10)")
 			(pintype "passive")
 		)
@@
 			(layers "B.Cu" "B.Mask" "B.Paste")
 			(roundrect_rratio 0.25)
-			(net "Net-(Q1-G)")
+			(net "Net-(ESP32s3-GPIO11)")
 			(pinfunction "G_1")
 			(pintype "input")
@@
 			(layers "B.Cu" "B.Mask" "B.Paste")
 			(roundrect_rratio 0.25)
-			(net "Net-(Q2-G)")
+			(net "Net-(ESP32s3-GPIO9)")
 			(pintype "passive")
 		)
@@
 		(width 0.4)
 		(layer "B.Cu")
-		(net "Net-(Q5-G)")
+		(net "Net-(ESP32s3-GPIO1)")
 	)
 	(segment
@@
 		(width 0.4)
 		(layer "B.Cu")
-		(net "Net-(Q5-G)")
+		(net "Net-(ESP32s3-GPIO1)")
 	)
 	(segment
@@
 		(width 0.4)
 		(layer "B.Cu")
-		(net "Net-(Q5-G)")
+		(net "Net-(ESP32s3-GPIO1)")
 	)
 	(segment
@@
 		(width 0.4)
 		(layer "B.Cu")
-		(net "Net-(Q5-G)")
+		(net "Net-(ESP32s3-GPIO1)")
 	)
 	(segment
@@
 		(width 0.4)
 		(layer "B.Cu")
-		(net "Net-(Q6-G)")
+		(net "Net-(ESP32s3-GPIO7)")
 	)
 	(segment
@@
 		(width 0.4)
 		(layer "B.Cu")
-		(net "Net-(Q6-G)")
+		(net "Net-(ESP32s3-GPIO7)")
 	)
 	(segment
@@
 		(width 0.4)
 		(layer "B.Cu")
-		(net "Net-(Q6-G)")
+		(net "Net-(ESP32s3-GPIO7)")
 	)
 	(segment
@@
 		(width 0.4)
 		(layer "B.Cu")
-		(net "Net-(Q6-G)")
+		(net "Net-(ESP32s3-GPIO7)")
 	)
 	(segment
@@
 		(width 0.4)
 		(layer "B.Cu")
-		(net "Net-(Q1-G)")
+		(net "Net-(ESP32s3-GPIO11)")
 	)
 	(segment
@@
 		(width 0.4)
 		(layer "B.Cu")
-		(net "Net-(Q1-G)")
+		(net "Net-(ESP32s3-GPIO11)")
 	)
 	(segment
@@
 		(width 0.4)
 		(layer "B.Cu")
-		(net "Net-(Q1-G)")
+		(net "Net-(ESP32s3-GPIO11)")
 	)
 	(segment
@@
 		(width 0.4)
 		(layer "B.Cu")
-		(net "Net-(Q1-G)")
+		(net "Net-(ESP32s3-GPIO11)")
 	)
 	(segment
@@
 		(width 0.4)
 		(layer "B.Cu")
-		(net "Net-(Q1-G)")
+		(net "Net-(ESP32s3-GPIO11)")
 	)
 	(segment
@@
 		(width 0.4)
 		(layer "B.Cu")
-		(net "Net-(Q4-G)")
+		(net "Net-(ESP32s3-GPIO10)")
 	)
 	(segment
@@
 		(width 0.4)
 		(layer "B.Cu")
-		(net "Net-(Q4-G)")
+		(net "Net-(ESP32s3-GPIO10)")
 	)
 	(segment
@@
 		(width 0.4)
 		(layer "B.Cu")
-		(net "Net-(Q4-G)")
+		(net "Net-(ESP32s3-GPIO10)")
 	)
 	(segment
@@
 		(width 0.4)
 		(layer "B.Cu")
-		(net "Net-(Q4-G)")
+		(net "Net-(ESP32s3-GPIO10)")
 	)
 	(segment
@@
 		(width 0.4)
 		(layer "B.Cu")
-		(net "Net-(Q4-G)")
+		(net "Net-(ESP32s3-GPIO10)")
 	)
 	(segment
@@
 		(width 0.4)
 		(layer "B.Cu")
-		(net "Net-(Q7-G)")
+		(net "Net-(ESP32s3-GPIO3)")
 	)
 	(segment
@@
 		(width 0.4)
 		(layer "B.Cu")
-		(net "Net-(Q7-G)")
+		(net "Net-(ESP32s3-GPIO3)")
 	)
 	(segment
@@
 		(width 0.4)
 		(layer "B.Cu")
-		(net "Net-(Q7-G)")
+		(net "Net-(ESP32s3-GPIO3)")
 	)
 	(segment
@@
 		(width 0.4)
 		(layer "B.Cu")
-		(net "Net-(Q7-G)")
+		(net "Net-(ESP32s3-GPIO3)")
 	)
 	(segment
@@
 		(width 0.4)
 		(layer "B.Cu")
-		(net "Net-(Q7-G)")
+		(net "Net-(ESP32s3-GPIO3)")
 	)
 	(segment
@@
 		(width 0.4)
 		(layer "B.Cu")
-		(net "Net-(Q3-G)")
+		(net "Net-(ESP32s3-GPIO13)")
 	)
 	(segment
@@
 		(width 0.4)
 		(layer "B.Cu")
-		(net "Net-(Q3-G)")
+		(net "Net-(ESP32s3-GPIO13)")
 	)
 	(segment
@@
 		(width 0.4)
 		(layer "B.Cu")
-		(net "Net-(Q3-G)")
+		(net "Net-(ESP32s3-GPIO13)")
 	)
 	(segment
@@
 		(width 0.4)
 		(layer "B.Cu")
-		(net "Net-(Q3-G)")
+		(net "Net-(ESP32s3-GPIO13)")
 	)
 	(segment
@@
 		(width 0.4)
 		(layer "B.Cu")
-		(net "Net-(Q3-G)")
+		(net "Net-(ESP32s3-GPIO13)")
 	)
 	(segment
@@
 		(width 0.4)
 		(layer "B.Cu")
-		(net "Net-(Q3-G)")
+		(net "Net-(ESP32s3-GPIO13)")
 	)
 	(segment
@@
 		(width 0.4)
 		(layer "B.Cu")
-		(net "Net-(Q2-G)")
+		(net "Net-(ESP32s3-GPIO9)")
 	)
 	(segment
@@
 		(width 0.4)
 		(layer "B.Cu")
-		(net "Net-(Q2-G)")
+		(net "Net-(ESP32s3-GPIO9)")
 	)
 	(segment
@@
 		(width 0.4)
 		(layer "B.Cu")
-		(net "Net-(Q2-G)")
+		(net "Net-(ESP32s3-GPIO9)")
 	)
 	(segment
@@
 		(width 0.4)
 		(layer "B.Cu")
-		(net "Net-(Q2-G)")
+		(net "Net-(ESP32s3-GPIO9)")
 	)
 	(segment
@@
 		(width 0.4)
 		(layer "B.Cu")
-		(net "Net-(Q2-G)")
+		(net "Net-(ESP32s3-GPIO9)")
 	)
 	(segment
@@
 		(width 0.4)
 		(layer "B.Cu")
-		(net "Net-(Q2-G)")
+		(net "Net-(ESP32s3-GPIO9)")
 	)
 	(segment
@@
 		(width 0.4)
 		(layer "B.Cu")
-		(net "Net-(Q2-G)")
+		(net "Net-(ESP32s3-GPIO9)")
 	)
 	(zone
